File: eagle/dip.sch (EAGLE design)
At the start: 9 parts

Commit message: inital V3 commit
Parts:
- removed JP6: M01PTH, SparkFun-Connectors:M01PTH
- added BAT1: (no value), SparkFun-Electromechanical:BATTERY12MM
- added R1, R2, R3: RESISTOR, thewknd:RESISTOR
- added S1: (no value), SparkFun-Electromechanical:TAC_SWITCHSMD
- added SJ1, SJ2: SOLDERJUMPERNO, SparkFun-Passives:SOLDERJUMPERNO
- JP1, JP2: value M20 -> M14; device SparkFun-Connectors:M20 -> SparkFun-Connectors:M14
- JP5: device SparkFun-Connectors:M03PTH -> SparkFun-Connectors:M05PTH
- JP8, JP9: value (none) -> M10"; device SparkFun-Connectors:M04PTH -> SparkFun-Connectors:M10"
Connections:
- removed net 3V3: JP2.18
- new net +3V3: JP2.12, JP7.2, R3.2, SJ1.2, SJ2.2
- new net N$2: R2.2, SJ1.1
- new net N$3: R1.2, SJ2.1
- net A0: now also JP2.2; no longer JP2.8
- net A1: now also JP2.3; no longer JP2.9
- net A10: now also JP5.4; no longer JP5.2
- net A11: now also JP5.5; no longer JP5.3
- net A2: now also JP2.4; no longer JP2.10
- net A3: now also JP2.5; no longer JP2.11
- net A4: now also JP2.6, R2.1; no longer JP2.12
- net A5: now also JP2.7, R1.1; no longer JP2.13
- net A6: now also JP2.8; no longer JP2.14
- net A7: now also JP2.9; no longer JP2.15
- net A8: now also JP2.10; no longer JP2.16
- net A9: now also JP2.11; no longer JP2.17
- net AGND: now also JP2.13; no longer JP2.19
- net AREF: now also JP5.3, JP9.6; no longer JP2.2, JP5.1
- net D0: now also JP1.13; no longer JP1.19
- net D1: now also JP1.12; no longer JP1.18
- net D10: now also JP1.3; no longer JP1.9
- net D11: now also JP1.2; no longer JP1.8
- net D12: now also JP1.1; no longer JP1.7
- net D13: now also JP2.1; no longer JP2.7
- net D2: now also JP1.11; no longer JP1.17
- net D24: now also JP8.10; no longer JP1.6
- net D25: now also JP8.9; no longer JP1.5
- net D26: now also JP8.8; no longer JP1.4
- net D27: now also JP8.7; no longer JP1.3
- net D28: now also JP8.6; no longer JP1.2
- net D29: now also JP8.5; no longer JP1.1
- net D3: now also JP1.10; no longer JP1.16
- net D4: now also JP1.9; no longer JP1.15
- net D5: now also JP1.8; no longer JP1.14
- net D6: now also JP1.7; no longer JP1.13
- net D7: now also JP1.6; no longer JP1.12
- net D8: now also JP1.5; no longer JP1.11
- net D9: now also JP1.4; no longer JP1.10
- net GND: now also BAT1.-, JP1.14, JP9.9, S1.3, S1.4; no longer JP1.20, JP2.5
- net PROG: now also JP9.5; no longer JP2.1
- net RESET: now also JP9.7, R3.1, S1.1, S1.2; no longer JP2.3
- net VBAT: now also BAT1.+, JP9.10; no longer JP2.6
- net VIN: now also JP2.14; no longer JP2.20
- net VUSB: now also JP5.1, JP9.8; no longer JP2.4, JP6.1
Other:
- note added: "Teensy 3.0 to breadboard adapter This work is licensed under a Creative Commons Attribution-ShareAlike 3.0 Unported License. http://creativecommons.org/licenses/by-sa/3.0/ (c) 2012, 2013 Jonas Niggli (thewknd)"
- note removed: "Teensy 3.0 to breadboard adapter This work is licensed under a Creative Commons Attribution-ShareAlike 3.0 Unported License. http://creativecommons.org/licenses/by-sa/3.0/ (c) 2012 Jonas Niggli (thewknd)"
- moved on the sheet: JP3, JP4, JP7

Commit message: new reset button
Parts:
- S1: value (none) -> SWITCH-PTH; device SparkFun-Electromechanical:TAC_SWITCHSMD -> thewknd:SWITCH-PTH
Changed lines of the file:
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@@
 <grid distance="0.1" unitdist="inch" unit="inch" style="lines" multiple="1" display="no" altdistance="0.01" altunitdist="inch" altunit="inch"/>
 <layers>
-<layer number="1" name="Top" color="4" fill="1" visible="no" active="no"/>
-<layer number="16" name="Bottom" color="1" fill="1" visible="no" active="no"/>
-<layer number="17" name="Pads" color="2" fill="1" visible="no" active="no"/>
-<layer number="18" name="Vias" color="2" fill="1" visible="no" active="no"/>
-<layer number="19" name="Unrouted" color="6" fill="1" visible="no" active="no"/>
-<layer number="20" name="Dimension" color="15" fill="1" visible="no" active="no"/>
-<layer number="21" name="tPlace" color="7" fill="1" visible="no" active="no"/>
-<layer number="22" name="bPlace" color="7" fill="1" visible="no" active="no"/>
-<layer number="23" name="tOrigins" color="15" fill="1" visible="no" active="no"/>
-<layer number="24" name="bOrigins" color="15" fill="1" visible="no" active="no"/>
-<layer number="25" name="tNames" color="7" fill="1" visible="no" active="no"/>
-<layer number="26" name="bNames" color="7" fill="1" visible="no" active="no"/>
-<layer number="27" name="tValues" color="7" fill="1" visible="no" active="no"/>
-<layer number="28" name="bValues" color="7" fill="1" visible="no" active="no"/>
+<layer number="1" name="Top" color="4" fill="1" visible="yes" active="no"/>
+<layer number="16" name="Bottom" color="1" fill="1" visible="yes" active="no"/>
+<layer number="17" name="Pads" color="2" fill="1" visible="yes" active="no"/>
+<layer number="18" name="Vias" color="2" fill="1" visible="yes" active="no"/>
+<layer number="19" name="Unrouted" color="6" fill="1" visible="yes" active="no"/>
+<layer number="20" name="Dimension" color="15" fill="1" visible="yes" active="no"/>
+<layer number="21" name="tPlace" color="7" fill="1" visible="yes" active="no"/>
+<layer number="22" name="bPlace" color="7" fill="1" visible="yes" active="no"/>
+<layer number="23" name="tOrigins" color="15" fill="1" visible="yes" active="no"/>
+<layer number="24" name="bOrigins" color="15" fill="1" visible="yes" active="no"/>
+<layer number="25" name="tNames" color="7" fill="1" visible="yes" active="no"/>
+<layer number="26" name="bNames" color="7" fill="1" visible="yes" active="no"/>
+<layer number="27" name="tValues" color="7" fill="1" visible="yes" active="no"/>
+<layer number="28" name="bValues" color="7" fill="1" visible="yes" active="no"/>
 <layer number="29" name="tStop" color="7" fill="3" visible="no" active="no"/>
 <layer number="30" name="bStop" color="7" fill="6" visible="no" active="no"/>
@@
 <layer number="35" name="tGlue" color="7" fill="4" visible="no" active="no"/>
 <layer number="36" name="bGlue" color="7" fill="5" visible="no" active="no"/>
-<layer number="37" name="tTest" color="7" fill="1" visible="no" active="no"/>
-<layer number="38" name="bTest" color="7" fill="1" visible="no" active="no"/>
+<layer number="37" name="tTest" color="7" fill="1" visible="yes" active="no"/>
+<layer number="38" name="bTest" color="7" fill="1" visible="yes" active="no"/>
 <layer number="39" name="tKeepout" color="4" fill="11" visible="no" active="no"/>
 <layer number="40" name="bKeepout" color="1" fill="11" visible="no" active="no"/>
@@
 <layer number="44" name="Drills" color="7" fill="1" visible="no" active="no"/>
 <layer number="45" name="Holes" color="7" fill="1" visible="no" active="no"/>
-<layer number="46" name="Milling" color="3" fill="1" visible="no" active="no"/>
-<layer number="47" name="Measures" color="7" fill="1" visible="no" active="no"/>
-<layer number="48" name="Document" color="7" fill="1" visible="no" active="no"/>
-<layer number="49" name="Reference" color="7" fill="1" visible="no" active="no"/>
-<layer number="50" name="dxf" color="7" fill="1" visible="no" active="no"/>
-<layer number="51" name="tDocu" color="7" fill="1" visible="no" active="no"/>
-<layer number="52" name="bDocu" color="7" fill="1" visible="no" active="no"/>
-<layer number="53" name="tGND_GNDA" color="7" fill="9" visible="no" active="no"/>
-<layer number="54" name="bGND_GNDA" color="1" fill="9" visible="no" active="no"/>
-<layer number="56" name="wert" color="7" fill="1" visible="no" active="no"/>
+<layer number="46" name="Milling" color="3" fill="1" visible="yes" active="no"/>
+<layer number="47" name="Measures" color="7" fill="1" visible="yes" active="no"/>
+<layer number="48" name="Document" color="7" fill="1" visible="yes" active="no"/>
+<layer number="49" name="Reference" color="7" fill="1" visible="yes" active="no"/>
+<layer number="50" name="dxf" color="7" fill="1" visible="yes" active="no"/>
+<layer number="51" name="tDocu" color="14" fill="1" visible="yes" active="no"/>
+<layer number="52" name="bDocu" color="7" fill="1" visible="yes" active="no"/>
+<layer number="53" name="tGND_GNDA" color="7" fill="9" visible="yes" active="no"/>
+<layer number="54" name="bGND_GNDA" color="1" fill="9" visible="yes" active="no"/>
+<layer number="56" name="wert" color="7" fill="1" visible="yes" active="no"/>
 <layer number="91" name="Nets" color="2" fill="1" visible="yes" active="yes"/>
 <layer number="92" name="Busses" color="1" fill="1" visible="yes" active="yes"/>
@@
 <part name="JP4" library="SparkFun-Connectors" deviceset="M07" device=""/>
 <part name="JP7" library="SparkFun-Connectors" deviceset="M05" device="PTH"/>
-<part name="S1" library="SparkFun-Electromechanical" deviceset="TAC_SWITCH" device="SMD"/>
+<part name="S1" library="thewknd" deviceset="SWITCH" device="-PTH"/>
 <part name="GND1" library="supply1" deviceset="GND" device=""/>
 <part name="BAT1" library="SparkFun-Electromechanical" deviceset="BATTERY" device="12MM"/>
@@
 <instance part="JP4" gate="G$1" x="109.22" y="165.1"/>
 <instance part="JP7" gate="G$1" x="73.66" y="119.38"/>
-<instance part="S1" gate="S" x="160.02" y="162.56"/>
+<instance part="S1" gate="G$1" x="160.02" y="162.56"/>
 <instance part="GND1" gate="1" x="170.18" y="152.4"/>
 <instance part="BAT1" gate="G$1" x="198.12" y="167.64"/>
@@
 </segment>
 <segment>
-<pinref part="S1" gate="S" pin="3"/>
-<pinref part="S1" gate="S" pin="4"/>
-<wire x1="165.1" y1="162.56" x2="165.1" y2="160.02" width="0.1524" layer="91"/>
+<pinref part="S1" gate="G$1" pin="4"/>
 <pinref part="GND1" gate="1" pin="GND"/>
 <wire x1="165.1" y1="160.02" x2="170.18" y2="160.02" width="0.1524" layer="91"/>
 <wire x1="170.18" y1="160.02" x2="170.18" y2="154.94" width="0.1524" layer="91"/>
-<junction x="165.1" y="160.02"/>
+<wire x1="170.18" y1="160.02" x2="170.18" y2="162.56" width="0.1524" layer="91"/>
+<junction x="170.18" y="160.02"/>
+<pinref part="S1" gate="G$1" pin="3"/>
+<wire x1="170.18" y1="162.56" x2="165.1" y2="162.56" width="0.1524" layer="91"/>
 </segment>
 <segment>
@@
 </segment>
 <segment>
-<pinref part="S1" gate="S" pin="2"/>
-<pinref part="S1" gate="S" pin="1"/>
-<wire x1="154.94" y1="160.02" x2="154.94" y2="162.56" width="0.1524" layer="91"/>
+<pinref part="S1" gate="G$1" pin="1"/>
 <wire x1="154.94" y1="162.56" x2="149.86" y2="162.56" width="0.1524" layer="91"/>
-<junction x="154.94" y="162.56"/>
 <label x="142.24" y="162.56" size="0.8128" layer="95" rot="R180" xref="yes"/>
 <wire x1="149.86" y1="162.56" x2="142.24" y2="162.56" width="0.1524" layer="91"/>
 <pinref part="R3" gate="G$1" pin="1"/>
 <junction x="149.86" y="162.56"/>
-</segment>
-</net>
+<pinref part="S1" gate="G$1" pin="2"/>
+<wire x1="154.94" y1="160.02" x2="149.86" y2="160.02" width="0.1524" layer="91"/>
+<wire x1="149.86" y1="160.02" x2="149.86" y2="162.56" width="0.1524" layer="91"/>
+</segment>
+</net>
